Commit message: Added long fingers

File: motoman/motoman_sda10f_support/urdf/sda10f_macro.xacro (robot description, xacro)
@@ -117,12 +117,14 @@
                 <child link="hand_left_palm" />
             </joint> -->
+<!--
         <xacro:s-model_articulated prefix="hand_right_">
             <origin xyz="0 0 0" rpy="0 0 0" />
         </xacro:s-model_articulated>
-        <joint name="hand_right_joint" type="fixed">
+    -->
+<!--         <joint name="hand_right_joint" type="fixed">
            <origin rpy="1.57079 0 2.87979" xyz="0 0 0.0797125"/>
                 <parent link="cylinder_hand_right" />
                 <child link="hand_right_palm" />
-            </joint>
+            </joint> -->
   <!--      <joint name="hand_right_joint" type="fixed">
             <origin rpy="-1.57079 0 0" xyz="0 0 -0.0684"/>

Commit message: tray_model added

File: motoman/motoman_sda10f_support/urdf/sda10f_macro.xacro (robot description, xacro)
@@ -25,5 +25,5 @@
 		<visual>
 			<geometry>
-				<cylinder length=".0743" radius=".06" />
+				<cylinder length=".04" radius=".06" />
 			</geometry>
 			<material name="ylw">
@@ -46,5 +46,5 @@
                 <parent link="hand_left_palm" />
                 <child link="camera_left" />
-        </joint>
+    </joint>
     <link name="robotiq_hand_wires_left">
 		<visual>
@@ -77,39 +77,22 @@
                 <child link="robotiq_force_wires_left" />
     </joint>
-<!--
-	<link name="ft_sensor_cable_box_left">
-		<visual>
-			<geometry>
-				<box size=".055 .055 .033" />
-			</geometry>
-		</visual>
-	</link>
-	<link name="ft_sensor_cable_box_right">
-		<visual>
-			<geometry>
-				<box size=".055 .055 .033" />
-			</geometry>
-		</visual>
-	</link>
--->
-        <joint name="hand_cylinder_joint_left" type="fixed">
-            <origin rpy="3.14159 0 3.14159" xyz="0 0 0"/>
-                <parent link="arm_left_link_tool0" />
-                <child link="cylinder_hand_left" />
-        </joint>
-        <joint name="hand_cylinder_joint_right" type="fixed">
-            <origin rpy="3.14159 0 3.14159" xyz="0 0 -.03125"/>
-                <parent link="arm_right_link_tool0" />
-                <child link="cylinder_hand_right" />
-        </joint>
-        <xacro:s-model_articulated prefix="hand_left_">
-            <origin xyz="0 0 0" rpy="0 0 0" />
-        </xacro:s-model_articulated>
-<!--.077475-->
-        <joint name="hand_left_joint" type="fixed">
-           <origin rpy="1.57079 0 -0.26180" xyz="0 0 0.0797125"/>
-                <parent link="cylinder_hand_left" />
-                <child link="hand_left_palm" />
-            </joint>
+	<joint name="hand_cylinder_joint_left" type="fixed">
+		<origin rpy="3.14159 0 3.14159" xyz="0 0 0"/>
+			<parent link="arm_left_link_tool0" />
+			<child link="cylinder_hand_left" />
+	</joint>
+	<joint name="hand_cylinder_joint_right" type="fixed">
+		<origin rpy="3.14159 0 3.14159" xyz="0 0 -.03125"/>
+			<parent link="arm_right_link_tool0" />
+			<child link="cylinder_hand_right" />
+	</joint>
+	<xacro:s-model_articulated prefix="hand_left_">
+		<origin xyz="0 0 0" rpy="0 0 0" />
+	</xacro:s-model_articulated>
+	<joint name="hand_left_joint" type="fixed">
+	   <origin rpy="1.57079 0 -0.26180" xyz="0 0 0.0797125"/>
+			<parent link="cylinder_hand_left" />
+			<child link="hand_left_palm" />
+	</joint>
     <!--    <joint name="hand_left_joint" type="fixed">
             <origin rpy="-1.57079 0 3.14159" xyz="0 0 -0.0684"/>
@@ -117,12 +100,49 @@
                 <child link="hand_left_palm" />
             </joint> -->
-        <xacro:s-model_articulated prefix="hand_right_">
+<!--        <xacro:s-model_articulated prefix="hand_right_">
             <origin xyz="0 0 0" rpy="0 0 0" />
         </xacro:s-model_articulated>
-        <joint name="hand_right_joint" type="fixed">
-           <origin rpy="1.57079 0 2.87979" xyz="0 0 0.0797125"/>
+-->
+	<link name="traybody_hand_right">
+		<visual>
+			<geometry>
+				<box size="0.19 .005 .50" />
+			</geometry>
+			<material name="pwkl">
+          			<color rgba=".8 .6 1 1"/>
+         		</material>
+		</visual>
+	</link>
+	<link name="trayhandle_hand_right">
+		<visual>
+			<geometry>
+				<box size="0.155 .165 .015" />
+			</geometry>
+			<material name="pwkl">
+          			<color rgba=".8 .6 1 1"/>
+         		</material>
+		</visual>
+	</link>
+	<joint name="hand_right_joint" type="fixed">
+			<origin rpy="0 0 0" xyz="0.0 -0.05 0.03"/>
+			<parent link="cylinder_hand_right" />
+			<child link="trayhandle_hand_right" />
+    </joint>
+	<joint name="tray_joint" type="fixed">
+			<origin rpy="0 0 0" xyz="0.0 -0.08 0.25"/>
+			<parent link="trayhandle_hand_right" />
+			<child link="traybody_hand_right" />
+    </joint>
+<!--
+			<origin rpy="0 0.523 0" xyz="0.20 0 0.25"/>
+			<origin rpy="0 0.7853975 0" xyz="0.20 0 0.25"/>
+			<origin rpy="0 1.047 0" xyz="0.30 0 0.03"/>
+			<origin rpy="0 1.309 0" xyz="0.20 0 0.20"/>
+			<origin rpy="0 1.57 0" xyz="0.25 0 0.095"/>
+			<joint name="hand_right_joint" type="fixed">
+				<origin rpy="1.57079 0 2.87979" xyz="0 0 0.0797125"/>
                 <parent link="cylinder_hand_right" />
                 <child link="hand_right_palm" />
-            </joint>
+            </joint> -->
   <!--      <joint name="hand_right_joint" type="fixed">
             <origin rpy="-1.57079 0 0" xyz="0 0 -0.0684"/>

Commit message: updated tray model now more accurate

File: motoman/motoman_sda10f_support/urdf/sda10f_macro.xacro (robot description, xacro)
@@ -25,5 +25,5 @@
 		<visual>
 			<geometry>
-				<cylinder length=".0743" radius=".06" />
+				<cylinder length=".05" radius=".06" />
 			</geometry>
 			<material name="ylw">
@@ -112,4 +112,34 @@
                 <child link="hand_left_palm" />
             </joint>
+	<link name="traybody_hand_right">
+		<visual>
+			<geometry>
+				<box size="0.19 .005 .50" />
+			</geometry>
+			<material name="pwkl">
+          			<color rgba=".8 .6 1 1"/>
+         		</material>
+		</visual>
+	</link>
+	<link name="trayhandle_hand_right">
+		<visual>
+			<geometry>
+				<box size="0.155 .165 .015" />
+			</geometry>
+			<material name="pwkl">
+          			<color rgba=".8 .6 1 1"/>
+         		</material>
+		</visual>
+	</link>
+	<joint name="hand_right_joint" type="fixed">
+			<origin rpy="0 0 3.14159" xyz="0.0 0.05 0.0325"/>
+			<parent link="cylinder_hand_right" />
+			<child link="trayhandle_hand_right" />
+    </joint>
+	<joint name="tray_joint" type="fixed">
+			<origin rpy="0 0 0" xyz="0.0 -0.08 0.25"/>
+			<parent link="trayhandle_hand_right" />
+			<child link="traybody_hand_right" />
+    </joint>
     <!--    <joint name="hand_left_joint" type="fixed">
             <origin rpy="-1.57079 0 3.14159" xyz="0 0 -0.0684"/>

Commit message: Updated the angle of the tray (30 degree tilt)

File: motoman/motoman_sda10f_support/urdf/sda10f_macro.xacro (robot description, xacro)
@@ -133,5 +133,5 @@
 	</link>
 	<joint name="hand_right_joint" type="fixed">
-			<origin rpy="0 0 3.14159" xyz="0.0 0.05 0.0325"/>
+			<origin rpy="0 0 2.623674" xyz="0.0 0.05 0.0325"/>
 			<parent link="cylinder_hand_right" />
 			<child link="trayhandle_hand_right" />

Commit message: current tray mount updated

File: motoman/motoman_sda10f_support/urdf/sda10f_macro.xacro (robot description, xacro)
@@ -133,5 +133,5 @@
 	</link>
 	<joint name="hand_right_joint" type="fixed">
-			<origin rpy="0 0 2.623674" xyz="0.0 0.05 0.0325"/>
+			<origin rpy="0 0 2.623674" xyz="0.025 0.046 0.0325"/>
 			<parent link="cylinder_hand_right" />
 			<child link="trayhandle_hand_right" />

Commit message: Head wire box added

File: motoman/motoman_sda10f_support/urdf/sda10f_macro.xacro (robot description, xacro)
@@ -142,4 +142,19 @@
 			<child link="traybody_hand_right" />
     </joint>
+    <link name="head_wire">
+		<visual>
+			<geometry>
+				<box size="0.1 0.2 0.07" />
+			</geometry>
+            <material name="pwkl">
+          		<color rgba=".8 0 1 1"/>
+         	</material>
+		</visual>
+	</link>
+	<joint name="head_wire_joint" type="fixed">
+			<origin rpy="0 0 0" xyz="0.1 0.0 0.45"/>
+			<parent link="torso_link_b1" />
+			<child link="head_wire" />
+    </joint>
     <!--    <joint name="hand_left_joint" type="fixed">
             <origin rpy="-1.57079 0 3.14159" xyz="0 0 -0.0684"/>

Commit message: updated collision box for new camera mount

File: motoman/motoman_sda10f_support/urdf/sda10f_macro.xacro (robot description, xacro)
@@ -32,8 +32,8 @@
 		</visual>
 	</link>
-    <link name="camera_left">
+  <link name="camera_left">
 		<visual>
 			<geometry>
-				<box size=".11 .025 .035" />
+				<box size=".12 .065 .04" />
 			</geometry>
             <material name="pwkl">
@@ -43,8 +43,8 @@
 	</link>
     <joint name="camera_joint_left" type="fixed">
-            <origin rpy="0 0 0" xyz="0 0 .083"/>
-                <parent link="hand_left_palm" />
-                <child link="camera_left" />
-        </joint>
+            <origin rpy="0 0 0" xyz="0 0.07 0.05"/>
+                <parent link="arm_left_link_tool0" />
+                <child link="camera_left" />``
+    </joint>
     <link name="robotiq_hand_wires_left">
 		<visual>

Commit message: Add back and side walls of tray to model
First pass, expect more commits for refinement. Must verify visually in
RVIZ

File: motoman/motoman_sda10f_support/urdf/sda10f_macro.xacro (robot description, xacro)
@@ -132,4 +132,34 @@
 		</visual>
 	</link>
+   <link name="traysidewall1_hand_right">
+      <visual>
+         <geometry>
+            <box size ="0.125 0.043 0.015" />
+         </geometry>
+         <material name="pwkl">
+          			<color rgba=".8 .6 1 1"/>
+         		</material>
+		</visual>
+	</link>
+   <link name="traysidewall2_hand_right">
+      <visual>
+         <geometry>
+            <box size ="0.125 0.043 0.015" />
+         </geometry>
+         <material name="pwkl">
+                   <color rgba=".8 .6 1 1"/>
+               </material>
+      </visual>
+   </link>
+   <link name="traybackwall_hand_right">
+      <visual>
+         <geometry>
+            <box size ="0.175 0.065 0.015" />
+         </geometry>
+         <material name="pwkl">
+                   <color rgba=".8 .6 1 1"/>
+               </material>
+      </visual>
+   </link>
 	<joint name="hand_right_joint" type="fixed">
 			<origin rpy="0 0 2.623674" xyz="0.025 0.046 0.0325"/>
@@ -142,4 +172,19 @@
 			<child link="traybody_hand_right" />
     </joint>
+   <joint name="tray_joint_side_wall_1" type="fixed">
+      <origin rpy="1.5707963 0 0" xyz="0 0.10 -0.12" />
+      <parent link="traybody_hand_right" />
+      <child link="traysidewall1_hand_right" />
+   </joint>
+   <joint name="tray_joint_side_wall_2" type="fixed">
+      <origin rpy="1.5707963 0 0" xyz="0 -0.10 -0.12" />
+      <parent link="traybody_hand_right" />
+      <child link="traysidewall2_hand_right" />
+   </joint>
+   <joint name="tray_joint_back_wall" type="fixed">
+      <origin rpy="1.5707963 1.5707963 0" xyz="0 0 -0.20" />
+      <parent link="traybody_hand_right" />
+      <child link="traybackwall_hand_right" />
+   </joint>
     <link name="head_wire">
 		<visual>

Commit message: 2nd try for tray model

File: motoman/motoman_sda10f_support/urdf/sda10f_macro.xacro (robot description, xacro)
@@ -173,15 +173,15 @@
     </joint>
    <joint name="tray_joint_side_wall_1" type="fixed">
-      <origin rpy="1.5707963 0 0" xyz="0 0.10 -0.12" />
+      <origin rpy="0 1.5707963 0" xyz="0 0.10 -0.12" />
       <parent link="traybody_hand_right" />
       <child link="traysidewall1_hand_right" />
    </joint>
    <joint name="tray_joint_side_wall_2" type="fixed">
-      <origin rpy="1.5707963 0 0" xyz="0 -0.10 -0.12" />
+      <origin rpy="0 1.5707963 0" xyz="0 -0.10 -0.12" />
       <parent link="traybody_hand_right" />
       <child link="traysidewall2_hand_right" />
    </joint>
    <joint name="tray_joint_back_wall" type="fixed">
-      <origin rpy="1.5707963 1.5707963 0" xyz="0 0 -0.20" />
+      <origin rpy="0 1.5707963 1.5707963" xyz="0 0 -0.20" />
       <parent link="traybody_hand_right" />
       <child link="traybackwall_hand_right" />

Commit message: 3rd try

File: motoman/motoman_sda10f_support/urdf/sda10f_macro.xacro (robot description, xacro)
@@ -173,15 +173,15 @@
     </joint>
    <joint name="tray_joint_side_wall_1" type="fixed">
-      <origin rpy="0 1.5707963 0" xyz="0 0.10 -0.12" />
+      <origin rpy="0 1.5707963 0" xyz="0.1 0 -0.17" />
       <parent link="traybody_hand_right" />
       <child link="traysidewall1_hand_right" />
    </joint>
    <joint name="tray_joint_side_wall_2" type="fixed">
-      <origin rpy="0 1.5707963 0" xyz="0 -0.10 -0.12" />
+      <origin rpy="0 1.5707963 0" xyz="-0.1 0 -0.17" />
       <parent link="traybody_hand_right" />
       <child link="traysidewall2_hand_right" />
    </joint>
    <joint name="tray_joint_back_wall" type="fixed">
-      <origin rpy="0 1.5707963 1.5707963" xyz="0 0 -0.20" />
+      <origin rpy="0 0 0" xyz="0 0 -0.25" />
       <parent link="traybody_hand_right" />
       <child link="traybackwall_hand_right" />

Commit message: 4th try!

File: motoman/motoman_sda10f_support/urdf/sda10f_macro.xacro (robot description, xacro)
@@ -155,5 +155,5 @@
       <visual>
          <geometry>
-            <box size ="0.175 0.065 0.015" />
+            <box size ="0.175 0.065 0.07" />
          </geometry>
          <material name="pwkl">
@@ -173,15 +173,15 @@
     </joint>
    <joint name="tray_joint_side_wall_1" type="fixed">
-      <origin rpy="0 1.5707963 0" xyz="0.1 0 -0.17" />
+      <origin rpy="0 1.5707963 0" xyz="0.085 -0.023 -0.17" />
       <parent link="traybody_hand_right" />
       <child link="traysidewall1_hand_right" />
    </joint>
    <joint name="tray_joint_side_wall_2" type="fixed">
-      <origin rpy="0 1.5707963 0" xyz="-0.1 0 -0.17" />
+      <origin rpy="0 1.5707963 0" xyz="-0.085 -0.023 -0.17" />
       <parent link="traybody_hand_right" />
       <child link="traysidewall2_hand_right" />
    </joint>
    <joint name="tray_joint_back_wall" type="fixed">
-      <origin rpy="0 0 0" xyz="0 0 -0.25" />
+      <origin rpy="0 0 0" xyz="0 -0.03 -0.21" />
       <parent link="traybody_hand_right" />
       <child link="traybackwall_hand_right" />

Commit message: updated motoman urdf

File: motoman/motoman_sda10f_support/urdf/sda10f_macro.xacro (robot description, xacro)
@@ -15,5 +15,5 @@
 		<visual>
 			<geometry>
-				<cylinder length=".0743" radius=".06" />
+				<cylinder length=".1638" radius=".06" />
 			</geometry>
 			<material name="ylw">
@@ -25,5 +25,5 @@
 		<visual>
 			<geometry>
-				<cylinder length=".0743" radius=".06" />
+				<cylinder length=".0625" radius=".06" />
 			</geometry>
 			<material name="ylw">
@@ -94,5 +94,5 @@
 -->
         <joint name="hand_cylinder_joint_left" type="fixed">
-            <origin rpy="3.14159 0 3.14159" xyz="0 0 0"/>
+            <origin rpy="3.14159 0 3.14159" xyz="0 0 -0.03125"/>
                 <parent link="arm_left_link_tool0" />
                 <child link="cylinder_hand_left" />
@@ -108,5 +108,5 @@
 <!--.077475-->
         <joint name="hand_left_joint" type="fixed">
-           <origin rpy="1.57079 0 -0.26180" xyz="0 0 0.0797125"/>
+           <origin rpy="1.57079 0 -0.26180" xyz="0 0 0.0819"/>
                 <parent link="cylinder_hand_left" />
                 <child link="hand_left_palm" />

Commit message: updated URDF for accurate hand offsets

File: motoman/motoman_sda10f_support/urdf/sda10f_macro.xacro (robot description, xacro)
@@ -43,5 +43,5 @@
 	</link>
     <joint name="camera_joint_left" type="fixed">
-            <origin rpy="0 0 0" xyz="0 0.07 0.02"/>
+            <origin rpy="0 0 0" xyz="0 0.07 -0.02"/>
                 <parent link="arm_left_link_tool0" />
                 <child link="camera_left" />``
@@ -155,5 +155,6 @@
       <visual>
          <geometry>
-            <box size ="0.175 0.065 0.07" />
+            <!-- <box size ="0.175 0.065 0.07" /> -->
+            <box size ="0.175 0.14 0.07" />
          </geometry>
          <material name="pwkl">
@@ -163,5 +164,6 @@
    </link>
 	<joint name="hand_right_joint" type="fixed">
-			<origin rpy="0 0 2.623674" xyz="0.025 0.046 0.0325"/>
+			<!-- <origin rpy="0 0 2.623674" xyz="0.025 0.046 0.0325"/> -->
+      <origin rpy="0 0 2.623674" xyz="0.025 0.046 0.040"/>
 			<parent link="cylinder_hand_right" />
 			<child link="trayhandle_hand_right" />
@@ -183,5 +185,6 @@
    </joint>
    <joint name="tray_joint_back_wall" type="fixed">
-      <origin rpy="0 0 0" xyz="0 -0.03 -0.21" />
+      <!-- <origin rpy="0 0 0" xyz="0 -0.03 -0.21" /> -->
+      <origin rpy="0 0 0" xyz="0 0 -0.21" />
       <parent link="traybody_hand_right" />
       <child link="traybackwall_hand_right" />

Commit message: updated collision model

File: motoman/motoman_sda10f_support/urdf/sda10f_macro.xacro (robot description, xacro)
@@ -77,4 +77,19 @@
                 <child link="robotiq_force_wires_left" />
     </joint>
+  <link name="torso_cylinder">
+    <visual>
+      <geometry>
+        <cylinder length="1" radius="0.15" />
+      </geometry>
+            <material name="pwkl">
+              <color rgba=".8 .8 1 1"/>
+          </material>
+    </visual>`
+  </link>
+  <joint name="torso_cylinder_joint" type="fixed">
+      <origin rpy="0 0 0" xyz="0.1 0 0.5"/>
+          <parent link="base_link" />
+          <child link="torso_cylinder" />
+  </joint>
 <!--
 	<link name="ft_sensor_cable_box_left">

Commit message: updated tray model in urdf

File: motoman/motoman_sda10f_support/urdf/sda10f_macro.xacro (robot description, xacro)
@@ -130,5 +130,5 @@
 		<visual>
 			<geometry>
-				<box size="0.19 .005 .50" />
+				<box size="0.20 .05 .50" />
 			</geometry>
 			<material name="pwkl">
@@ -140,5 +140,5 @@
 		<visual>
 			<geometry>
-				<box size="0.155 .165 .015" />
+				<box size="0.16 .17 .03" />
 			</geometry>
 			<material name="pwkl">
