Commit message: Changed step size

File: motoman/motoman_sda10f_support/urdf/common_torso_macro.xacro (robot description, xacro)
@@ -40,5 +40,5 @@
 		</link>
 		<link name="${prefix}link_b2">
-			<visual>
+<!-- 			<visual>
 				<origin rpy="0 0 0" xyz="0 0 0"/>
 				<geometry>
@@ -55,5 +55,5 @@
 				</geometry>
 				<material name="yellow"/>
-			</collision>
+			</collision> -->
 		</link>
 		<!-- joint list -->
