Commit message: updated URDF with new camera position

File: motoman/motoman_sda10f_support/urdf/arm_macro.xacro (robot description, xacro)
@@ -141,5 +141,5 @@
 			<origin xyz="0 -0.0085 -0.181" rpy="-1.57 0 0"/>
 			<axis xyz="0 0 ${reflect}" />
-			<limit lower="-2.36" upper="2.36" effort="0" velocity="2.95" />
+			<limit lower="-2.3" upper="2.3" effort="0" velocity="2.95" />
 		</joint>
 		<joint name="${prefix}joint_5_r" type="revolute">

File: motoman/motoman_sda10f_support/urdf/sda10f_macro.xacro (robot description, xacro)
@@ -43,5 +43,5 @@
 	</link>
     <joint name="camera_joint_left" type="fixed">
-            <origin rpy="0 0 0" xyz="0 0.07 0.05"/>
+            <origin rpy="0 0 0" xyz="0 0.07 0.02"/>
                 <parent link="arm_left_link_tool0" />
                 <child link="camera_left" />``

Commit message: Fixed joint offsets

File: motoman/motoman_sda10f_support/urdf/arm_macro.xacro (robot description, xacro)
@@ -132,5 +132,5 @@
 			<parent link="${prefix}link_2_l"/>
 			<child link="${prefix}link_3_e"/>
-			<origin xyz="0 0.1690 -0.0454" rpy="1.57 0 0"/>
+			<origin xyz="0 0.1790 -0.0454" rpy="1.57 0 0"/>
 			<axis xyz="0 0 ${-reflect}" />
 			<limit lower="-2.95" upper="2.95" effort="0" velocity="2.95" />
@@ -139,5 +139,5 @@
 			<parent link="${prefix}link_3_e"/>
 			<child link="${prefix}link_4_u"/>
-			<origin xyz="0 -0.0085 -0.181" rpy="-1.57 0 0"/>
+			<origin xyz="0 -0.0165 -0.181" rpy="-1.57 0 0"/>
 			<axis xyz="0 0 ${reflect}" />
 			<limit lower="-2.3" upper="2.3" effort="0" velocity="2.95" />
@@ -146,5 +146,5 @@
 			<parent link="${prefix}link_4_u"/>
 			<child link="${prefix}link_5_r"/>
-			<origin xyz="0 0.1936 0.0155" rpy="1.57 0 0"/>
+			<origin xyz="0 0.2026 0.0155" rpy="1.57 0 0"/>
 			<axis xyz="0 0 ${reflect}" />
 			<limit lower="-3.13" upper="3.13" effort="0" velocity="3.48" />
@@ -153,5 +153,5 @@
 			<parent link="${prefix}link_5_r"/>
 			<child link="${prefix}link_6_b"/>
-			<origin xyz="0 0.0080 -0.155" rpy="-1.57 0 0"/>
+			<origin xyz="0 0.0170 -0.155" rpy="-1.57 0 0"/>
 			<axis xyz="0 0 ${reflect}" />
 			<limit lower="-1.90" upper="1.90" effort="0" velocity="3.48" />
